File: Raspberry Pi HAT EEPROM/KiCad Design/Raspberry Pi HAT EEPROM.kicad_sch (KiCad schematic)
At the start: 0 parts

Commit message: Notionally complete through PA
Parts:
- added C14: 100n, Capacitor_SMD:C_0603_1608Metric, symbol Device:C_Small
- added R11: 47kΩ, Resistor_SMD:R_0603_1608Metric, symbol Device:R_US
- added R12, R14: 3.9K, Resistor_SMD:R_0603_1608Metric, symbol Device:R_US
- added R13: 0Ω, Resistor_SMD:R_0603_1608Metric, symbol Device:R_US
- added U2: 24LC128, Package_SO:SOIC-8_3.9x4.9mm_P1.27mm, symbol Memory_EEPROM:24LC128
Connections:
- new net: R11.1, R13.1, U2.7 (WP)
- new net ID_3V3: C14.2, R12.1, R13.2, R14.1, U2.8 (VCC)
- new net ID_GND: C14.1, R11.2, U2.1 (A0), U2.2 (A1), U2.3 (A2), U2.4 (GND)
- new net ID_SCL: R14.2, U2.6 (SCL)
- new net ID_SDA: R12.2, U2.5 (SDA)
Other:
- removed sheet ID EEPROM
- removed sheet Raspberry Pi Header
- note added: "ID_SD and ID_SC PINS: These pins are reserved for HAT ID EEPROM. At boot time this I2C interface will be interrogated to look for an EEPROM that identifes the attached board and allows automagic setup of the GPIOs (and optionally, Linux drivers). Bridging R3 pads (NP) enables write protection. DO NOT USE these pins for anything other than attaching an I2C ID EEPROM. Leave unconnected if ID EEPROM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"
- note removed: "Additional pin functions: https://pinout.xyz/"
- title: Raspberry Pi µHAT -> Raspberry Pi HAT+ EEPROM
