File: WSPR Si5153 RF Chain/Components/27 MHz TCXO Block/KiCad Design/27 MHz TCXO Block.kicad_sch (KiCad schematic)
At the start: 9 parts, among them Y1 ATX-11-F-27.000MHZ-F05-T

Commit message: Notionally complete through PA
Parts:
- C2, C3, C4: footprint Capacitor_SMD:C_0201_0603Metric -> Capacitor_SMD:C_0603_1608Metric
- R3: renamed from R5; footprint Resistor_SMD:R_0201_0603Metric -> Resistor_SMD:R_0603_1608Metric
- R4: renamed from R6; footprint Resistor_SMD:R_0201_0603Metric -> Resistor_SMD:R_0603_1608Metric
- TP1, TP2: footprint (none) -> TestPoint:TestPoint_2Pads_Pitch2.54mm_Drill0.8mm
Connections:
- net XTAL_GND: now also C2.1, C3.1; no longer C2.2, C3.2
- net at FB1.1, Y1.4 (Vcc): now also C2.2, C3.2; no longer C2.1, C3.1
Other:
- note removed: "27MHz TCXO Circuit"
- moved on the sheet: C2
Changed lines of the file:
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@@
 	(title_block
 		(title "27 MHz TCXO Block")
-		(date "2026-02-04")
+		(date "2026-02-14")
 		(rev "0")
 		(company "Lee C. Bussy [AA0NT]")
-	)
-	(text "27MHz TCXO Circuit"
-		(exclude_from_sim no)
-		(at 133.858 57.658 0)
-		(effects
-			(font
-				(size 1.905 1.905)
-				(thickness 0.381)
-				(bold yes)
-			)
-		)
 	)
 	(text "The TCXO and its decoupling capacitors are clustered tightly.\nThe island is fed from the main 3V3 rail through a ferrite\nbead. Noise from the rest of the board (Pi GPIO, SPI, switching\nregulators) is attenuated before reaching the TCXO.\n\nGround returns go directly into a solid ground plane.\n\nThis improves frequency stability and minimizes phase noise\nmodulation.\n\nR2 is 0 Ω default, stuff 22 Ω if trace > ~25-50 mm."
@@
 	(wire
 		(pts
-			(xy 139.7 83.82) (xy 137.16 83.82)
-		)
-		(stroke
-			(width 0)
-			(type default)
-		)
-	)
-	(wire
-		(pts
 			(xy 129.54 85.09) (xy 129.54 83.82)
 		)
@@
 		(pts
 			(xy 144.78 83.82) (xy 146.05 83.82)
+		)
+		(stroke
+			(width 0)
+			(type default)
+		)
+	)
+	(wire
+		(pts
+			(xy 137.16 83.82) (xy 139.7 83.82)
 		)
 		(stroke
@@
 			)
 		)
-		(property "Footprint" ""
+		(property "Footprint" "TestPoint:TestPoint_2Pads_Pitch2.54mm_Drill0.8mm"
 			(at 165.1 97.79 0)
 			(effects
@@
 				)
 			)
-			(project "WSPR Si5351 RF Chain"
+			(project "27 MHz TCXO Block"
+				(path "/b45cd213-f13d-41d6-8d12-d5cd52542809"
+					(reference "TP2")
+					(unit 1)
+				)
+			)
+			(project "Wsprry_Pi_uHAT"
 				(path "/e63e39d7-6ac0-4ffd-8aa3-1841a4541b55/262a9111-a0c2-4bdb-b21f-e33adb0241de/42ba523c-9f36-4add-9ea4-d17afe81c991"
 					(reference "TP2")
@@
 	(symbol
 		(lib_id "Device:C")
-		(at 129.54 80.01 180)
+		(at 129.54 80.01 0)
 		(unit 1)
 		(exclude_from_sim no)
@@
 		(dnp no)
 		(property "Reference" "C2"
-			(at 126.238 80.01 0)
+			(at 130.81 82.042 0)
 			(effects
 				(font
@@
 		)
 		(property "Value" "0.1uF"
-			(at 133.096 82.55 0)
-			(effects
-				(font
-					(size 1.27 1.27)
-				)
-			)
-		)
-		(property "Footprint" "Capacitor_SMD:C_0201_0603Metric"
-			(at 128.5748 76.2 0)
+			(at 127 77.978 0)
+			(effects
+				(font
+					(size 1.27 1.27)
+				)
+			)
+		)
+		(property "Footprint" "Capacitor_SMD:C_0603_1608Metric"
+			(at 130.5052 83.82 0)
 			(effects
 				(font
@@
 				)
 			)
-			(project "WSPR Si5351 RF Chain"
+			(project "Wsprry_Pi_uHAT"
 				(path "/e63e39d7-6ac0-4ffd-8aa3-1841a4541b55/262a9111-a0c2-4bdb-b21f-e33adb0241de/42ba523c-9f36-4add-9ea4-d17afe81c991"
 					(reference "C2")
@@
 			)
 		)
-		(property "Footprint" ""
+		(property "Footprint" "TestPoint:TestPoint_2Pads_Pitch2.54mm_Drill0.8mm"
 			(at 139.7 97.79 0)
 			(effects
@@
 				)
 			)
-			(project "WSPR Si5351 RF Chain"
+			(project "27 MHz TCXO Block"
+				(path "/b45cd213-f13d-41d6-8d12-d5cd52542809"
+					(reference "TP1")
+					(unit 1)
+				)
+			)
+			(project "Wsprry_Pi_uHAT"
 				(path "/e63e39d7-6ac0-4ffd-8aa3-1841a4541b55/262a9111-a0c2-4bdb-b21f-e33adb0241de/42ba523c-9f36-4add-9ea4-d17afe81c991"
 					(reference "TP1")
-					(unit 1)
-				)
-			)
-		)
-	)
-	(symbol
-		(lib_id "Device:C")
-		(at 137.16 80.01 180)
-		(unit 1)
-		(exclude_from_sim no)
-		(in_bom yes)
-		(on_board yes)
-		(dnp no)
-		(property "Reference" "C3"
-			(at 133.858 80.01 0)
-			(effects
-				(font
-					(size 1.27 1.27)
-				)
-			)
-		)
-		(property "Value" "1.0uF"
-			(at 140.716 82.55 0)
-			(effects
-				(font
-					(size 1.27 1.27)
-				)
-				(hide yes)
-			)
-		)
-		(property "Footprint" "Capacitor_SMD:C_0201_0603Metric"
-			(at 136.1948 76.2 0)
-			(effects
-				(font
-					(size 1.27 1.27)
-				)
-				(hide yes)
-			)
-		)
-		(property "Datasheet" "~"
-			(at 137.16 80.01 0)
-			(effects
-				(font
-					(size 1.27 1.27)
-				)
-				(hide yes)
-			)
-		)
-		(property "Description" "Unpolarized capacitor"
-			(at 137.16 80.01 0)
-			(effects
-				(font
-					(size 1.27 1.27)
-				)
-				(hide yes)
-			)
-		)
-		(pin "1"
-		)
-		(pin "2"
-		)
-		(instances
-			(project "WSPR Si5351 RF Chain"
-				(path "/ac78b79f-d9c0-46e3-b029-91bb1924b198/42ba523c-9f36-4add-9ea4-d17afe81c991"
-					(reference "C2")
-					(unit 1)
-				)
-			)
-			(project "Untitled"
-				(path "/b45cd213-f13d-41d6-8d12-d5cd52542809"
-					(reference "C2")
-					(unit 1)
-				)
-			)
-			(project "WSPR Si5351 RF Chain"
-				(path "/e63e39d7-6ac0-4ffd-8aa3-1841a4541b55/262a9111-a0c2-4bdb-b21f-e33adb0241de/42ba523c-9f36-4add-9ea4-d17afe81c991"
-					(reference "C3")
 					(unit 1)
 				)
@@
 			)
 		)
-		(property "Footprint" "Capacitor_SMD:C_0201_0603Metric"
+		(property "Footprint" "Capacitor_SMD:C_0603_1608Metric"
 			(at 156.21 91.7448 0)
 			(effects
@@
 				)
 			)
-			(project "WSPR Si5351 RF Chain"
+			(project "Wsprry_Pi_uHAT"
 				(path "/e63e39d7-6ac0-4ffd-8aa3-1841a4541b55/262a9111-a0c2-4bdb-b21f-e33adb0241de/42ba523c-9f36-4add-9ea4-d17afe81c991"
 					(reference "C4")
@@
 				)
 			)
-			(project "WSPR Si5351 RF Chain"
+			(project "Wsprry_Pi_uHAT"
 				(path "/e63e39d7-6ac0-4ffd-8aa3-1841a4541b55/262a9111-a0c2-4bdb-b21f-e33adb0241de/42ba523c-9f36-4add-9ea4-d17afe81c991"
 					(reference "FB1")
@@
 		(on_board yes)
 		(dnp no)
-		(property "Reference" "R5"
+		(property "Reference" "R3"
 			(at 143.51 90.17 90)
 			(effects
@@
 			)
 		)
-		(property "Footprint" "Resistor_SMD:R_0201_0603Metric"
+		(property "Footprint" "Resistor_SMD:R_0603_1608Metric"
 			(at 143.764 91.694 90)
 			(effects
@@
 				)
 			)
-			(project "WSPR Si5351 RF Chain"
+			(project "Wsprry_Pi_uHAT"
 				(path "/e63e39d7-6ac0-4ffd-8aa3-1841a4541b55/262a9111-a0c2-4bdb-b21f-e33adb0241de/42ba523c-9f36-4add-9ea4-d17afe81c991"
-					(reference "R5")
+					(reference "R3")
 					(unit 1)
 				)
@@
 		(on_board yes)
 		(dnp no)
-		(property "Reference" "R6"
+		(property "Reference" "R4"
 			(at 161.29 90.17 90)
 			(effects
@@
 			)
 		)
-		(property "Footprint" "Resistor_SMD:R_0201_0603Metric"
+		(property "Footprint" "Resistor_SMD:R_0603_1608Metric"
 			(at 161.544 91.694 90)
 			(effects
@@
 				)
 			)
-			(project "WSPR Si5351 RF Chain"
+			(project "Wsprry_Pi_uHAT"
 				(path "/e63e39d7-6ac0-4ffd-8aa3-1841a4541b55/262a9111-a0c2-4bdb-b21f-e33adb0241de/42ba523c-9f36-4add-9ea4-d17afe81c991"
-					(reference "R6")
+					(reference "R4")
+					(unit 1)
+				)
+			)
+		)
+	)
+	(symbol
+		(lib_id "Device:C")
+		(at 137.16 80.01 0)
+		(unit 1)
+		(exclude_from_sim no)
+		(in_bom yes)
+		(on_board yes)
+		(dnp no)
+		(property "Reference" "C3"
+			(at 138.43 82.042 0)
+			(effects
+				(font
+					(size 1.27 1.27)
+				)
+			)
+		)
+		(property "Value" "1.0uF"
+			(at 134.366 77.978 0)
+			(effects
+				(font
+					(size 1.27 1.27)
+				)
+			)
+		)
+		(property "Footprint" "Capacitor_SMD:C_0603_1608Metric"
+			(at 138.1252 83.82 0)
+			(effects
+				(font
+					(size 1.27 1.27)
+				)
+				(hide yes)
+			)
+		)
+		(property "Datasheet" "~"
+			(at 137.16 80.01 0)
+			(effects
+				(font
+					(size 1.27 1.27)
+				)
+				(hide yes)
+			)
+		)
+		(property "Description" "Unpolarized capacitor"
+			(at 137.16 80.01 0)
+			(effects
+				(font
+					(size 1.27 1.27)
+				)
+				(hide yes)
+			)
+		)
+		(pin "1"
+		)
+		(pin "2"
+		)
+		(instances
+			(project "Wsprry_Pi_uHAT"
+				(path "/e63e39d7-6ac0-4ffd-8aa3-1841a4541b55/262a9111-a0c2-4bdb-b21f-e33adb0241de/42ba523c-9f36-4add-9ea4-d17afe81c991"
+					(reference "C3")
 					(unit 1)
 				)
@@
 				)
 			)
-			(project "WSPR Si5351 RF Chain"
+			(project "Wsprry_Pi_uHAT"
 				(path "/e63e39d7-6ac0-4ffd-8aa3-1841a4541b55/262a9111-a0c2-4bdb-b21f-e33adb0241de/42ba523c-9f36-4add-9ea4-d17afe81c991"
 					(reference "Y1")
@@
 		(dnp no)
 		(fields_autoplaced yes)
-		(property "Reference" "#FLG07"
+		(property "Reference" "#FLG06"
 			(at 127.635 83.82 0)
 			(effects
@@
 		)
 		(instances
+			(project "WSPR Si5351 RF Chain"
+				(path "/ac78b79f-d9c0-46e3-b029-91bb1924b198/42ba523c-9f36-4add-9ea4-d17afe81c991"
+					(reference "#FLG0101")
+					(unit 1)
+				)
+			)
+			(project "27 MHz TCXO Block"
+				(path "/b45cd213-f13d-41d6-8d12-d5cd52542809"
+					(reference "#FLG01")
+					(unit 1)
+				)
+			)
 			(project ""
 				(path "/e63e39d7-6ac0-4ffd-8aa3-1841a4541b55/262a9111-a0c2-4bdb-b21f-e33adb0241de/42ba523c-9f36-4add-9ea4-d17afe81c991"
-					(reference "#FLG07")
-					(unit 1)
-				)
-			)
-		)
-	)
+					(reference "#FLG06")
+					(unit 1)
+				)
+			)
+		)
+	)
+	(sheet_instances
+		(path "/"
+			(page "1")
+		)
+	)
+	(embedded_fonts no)
 )
