File: WSPR Si5153 RF Chain/Components/3dB Pi Pad/KiCad Design/3dB Pad.kicad_sch (KiCad schematic)
At the start: 4 parts

Commit message: Notionally complete through PA
Parts:
- added TP3: TP_PAD_OUT, TestPoint:TestPoint_2Pads_Pitch2.54mm_Drill0.8mm, symbol Connector:TestPoint_2Pole
- C13: renamed from C18; value 10nF -> 0.1F; footprint Capacitor_SMD:C_0805_2012Metric -> Capacitor_SMD:C_0603_1608Metric
- R10: renamed from R18; value 150Ω -> 292Ω
- R8: renamed from R16; value 150Ω -> 292Ω
- R9: renamed from R17; value 37.4Ω -> 17.6Ω
Connections:
- net PAD_GND: now also TP3.2
- net BUFF_IN renamed CLOCK_IN
- net PAD_OUT renamed 3DB_PAD_OUT
- net 3DB_PAD_OUT: now also TP3.1
Other:
- note removed: "6dB Pi Pad"
- note removed: "We can drop to 3 dB if needed (Rshunt ≈ 292 Ω, Rseries ≈ 17.6 Ω)"
- moved on the sheet: C13, R10, R8, R9
