File: WSPR Si5153 RF Chain/Components/Broadband MMIC Gain Block/KiCad Design/Broadband_MMIC_Gain_Block.kicad_sch (KiCad schematic)
At the start: 9 parts, among them U2 GVA-84

Commit message: Notionally complete through PA
Parts:
- C10: renamed from C14; footprint Capacitor_SMD:C_0805_2012Metric -> Capacitor_SMD:C_0603_1608Metric
- C11: renamed from C15; footprint Capacitor_SMD:C_0805_2012Metric -> Capacitor_SMD:C_0603_1608Metric
- C12: renamed from C17; footprint Capacitor_SMD:C_0805_2012Metric -> Capacitor_SMD:C_1206_3216Metric
- C8: renamed from C13; footprint Capacitor_SMD:C_0805_2012Metric -> Capacitor_SMD:C_0603_1608Metric
- C9: renamed from C16; value 1µF -> 1.0µF; footprint Capacitor_SMD:C_0805_2012Metric -> Capacitor_SMD:C_0603_1608Metric
- L1: value 10µH -> 2.2µH; footprint Inductor_SMD:L_1206_3216Metric -> Inductor_SMD:L_0805_2012Metric
- R7: renamed from R15; value 10Ω -> 0Ω
- renumbered U2 to U1
Connections:
- net PLPF_IN renamed PAD_IN
Other:
- note added: "Pins 2 & 4 (ground pad)must be stitched to ground plane with vias. Place 0.1µF and 1.0µf within 3 mm of bias pin."
- note removed: "Broadband MMIC gain-block driver (gain varies with frequency)"
- note removed: "Pins 2 & 4 must be stitched to ground plane with vias. Place C2/C3 within 3 mm of bias pin."
- moved on the sheet: C10, C12, C9, FB3
