File: WSPR Si5153 RF Chain/Components/Si5351 Clock Generator Circuit/KiCad Design/Si5351 Clock Generator Circuit.kicad_sch (KiCad schematic)
At the start: 7 parts, among them Y2 Si5351A-B-GT

Commit message: Notionally complete through PA
Parts:
- C5, C6, C7: footprint (none) -> Capacitor_SMD:C_0603_1608Metric
- FB2: footprint (none) -> Inductor_SMD:L_0603_1608Metric
- R5: renamed from R7; footprint (none) -> Resistor_SMD:R_0603_1608Metric
- R6: renamed from R8; footprint (none) -> Resistor_SMD:R_0603_1608Metric
Changed lines of the file:
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@@
 	(title_block
 		(title "Si5351 Clock Generator Circuit")
-		(date "2026-02-03")
+		(date "2026-02-14")
 		(rev "0")
 		(company "Lee C. Bussy [AA0NT]")
@@
 	(wire
 		(pts
+			(xy 139.7 119.38) (xy 139.7 118.11)
+		)
+		(stroke
+			(width 0)
+			(type default)
+		)
+	)
+	(wire
+		(pts
 			(xy 119.38 110.49) (xy 127 110.49)
 		)
@@
 	(wire
 		(pts
+			(xy 125.73 97.79) (xy 127 97.79)
+		)
+		(stroke
+			(width 0)
+			(type default)
+		)
+	)
+	(wire
+		(pts
 			(xy 142.24 91.44) (xy 143.51 91.44)
 		)
@@
 		(pts
 			(xy 139.7 91.44) (xy 142.24 91.44)
-		)
-		(stroke
-			(width 0)
-			(type default)
-		)
-	)
-	(wire
-		(pts
-			(xy 125.73 97.79) (xy 127 97.79)
-		)
-		(stroke
-			(width 0)
-			(type default)
-		)
-	)
-	(wire
-		(pts
-			(xy 139.7 118.11) (xy 139.7 119.38)
 		)
 		(stroke
@@
 		(on_board yes)
 		(dnp no)
-		(property "Reference" "R7"
+		(property "Reference" "R5"
 			(at 120.65 116.84 0)
 			(effects
@@
 			)
 		)
-		(property "Footprint" ""
+		(property "Footprint" "Resistor_SMD:R_0603_1608Metric"
 			(at 120.396 118.364 90)
 			(effects
@@
 				)
 			)
-			(project "WSPR Si5351 RF Chain"
+			(project "Wsprry_Pi_uHAT"
 				(path "/e63e39d7-6ac0-4ffd-8aa3-1841a4541b55/262a9111-a0c2-4bdb-b21f-e33adb0241de/24e78a99-bad3-4a7d-9156-152997ea8218"
-					(reference "R7")
+					(reference "R5")
 					(unit 1)
 				)
@@
 			)
 		)
-		(property "Footprint" ""
+		(property "Footprint" "Capacitor_SMD:C_0603_1608Metric"
 			(at 128.27 92.4052 0)
 			(effects
@@
 		)
 		(instances
+			(project "WSPR Si5351 RF Chain"
+				(path "/ac78b79f-d9c0-46e3-b029-91bb1924b198/24e78a99-bad3-4a7d-9156-152997ea8218"
+					(reference "C?")
+					(unit 1)
+				)
+			)
+			(project "Si5351 Clock Generator Circuit"
+				(path "/dfe3e9ed-5269-4fae-b6d1-95c9618d8979"
+					(reference "C1")
+					(unit 1)
+				)
+			)
 			(project "Wsprry_Pi_uHAT"
 				(path "/e63e39d7-6ac0-4ffd-8aa3-1841a4541b55/262a9111-a0c2-4bdb-b21f-e33adb0241de/24e78a99-bad3-4a7d-9156-152997ea8218"
@@
 			)
 		)
-		(property "Footprint" ""
+		(property "Footprint" "Inductor_SMD:L_0603_1608Metric"
 			(at 140.462 81.28 90)
 			(effects
@@
 				)
 			)
-			(project "WSPR Si5351 RF Chain"
+			(project "Wsprry_Pi_uHAT"
 				(path "/e63e39d7-6ac0-4ffd-8aa3-1841a4541b55/262a9111-a0c2-4bdb-b21f-e33adb0241de/24e78a99-bad3-4a7d-9156-152997ea8218"
 					(reference "FB2")
@@
 			)
 		)
-		(property "Footprint" ""
+		(property "Footprint" "Capacitor_SMD:C_0603_1608Metric"
 			(at 151.13 90.4748 0)
 			(effects
@@
 				)
 			)
-			(project "WSPR Si5351 RF Chain"
+			(project "Wsprry_Pi_uHAT"
 				(path "/e63e39d7-6ac0-4ffd-8aa3-1841a4541b55/262a9111-a0c2-4bdb-b21f-e33adb0241de/24e78a99-bad3-4a7d-9156-152997ea8218"
 					(reference "C7")
@@
 		(dnp no)
 		(fields_autoplaced yes)
-		(property "Reference" "#FLG08"
+		(property "Reference" "#FLG07"
 			(at 139.7 89.535 0)
 			(effects
@@
 		)
 		(instances
+			(project "WSPR Si5351 RF Chain"
+				(path "/ac78b79f-d9c0-46e3-b029-91bb1924b198/24e78a99-bad3-4a7d-9156-152997ea8218"
+					(reference "#FLG0102")
+					(unit 1)
+				)
+			)
+			(project "Si5351 Clock Generator Circuit"
+				(path "/dfe3e9ed-5269-4fae-b6d1-95c9618d8979"
+					(reference "#FLG01")
+					(unit 1)
+				)
+			)
 			(project ""
 				(path "/e63e39d7-6ac0-4ffd-8aa3-1841a4541b55/262a9111-a0c2-4bdb-b21f-e33adb0241de/24e78a99-bad3-4a7d-9156-152997ea8218"
-					(reference "#FLG08")
+					(reference "#FLG07")
 					(unit 1)
 				)
@@
 			)
 		)
-		(property "Footprint" ""
+		(property "Footprint" "Capacitor_SMD:C_0603_1608Metric"
 			(at 151.13 85.3948 0)
 			(effects
@@
 				)
 			)
-			(project "WSPR Si5351 RF Chain"
+			(project "Wsprry_Pi_uHAT"
 				(path "/e63e39d7-6ac0-4ffd-8aa3-1841a4541b55/262a9111-a0c2-4bdb-b21f-e33adb0241de/24e78a99-bad3-4a7d-9156-152997ea8218"
 					(reference "C6")
@@
 				)
 			)
-			(project "WSPR Si5351 RF Chain"
+			(project "Wsprry_Pi_uHAT"
 				(path "/e63e39d7-6ac0-4ffd-8aa3-1841a4541b55/262a9111-a0c2-4bdb-b21f-e33adb0241de/24e78a99-bad3-4a7d-9156-152997ea8218"
 					(reference "Y2")
@@
 		(on_board yes)
 		(dnp no)
-		(property "Reference" "R8"
+		(property "Reference" "R6"
 			(at 126.746 116.84 0)
 			(effects
@@
 			)
 		)
-		(property "Footprint" ""
+		(property "Footprint" "Resistor_SMD:R_0603_1608Metric"
 			(at 126.746 118.364 90)
 			(effects
@@
 				)
 			)
-			(project "WSPR Si5351 RF Chain"
+			(project "Wsprry_Pi_uHAT"
 				(path "/e63e39d7-6ac0-4ffd-8aa3-1841a4541b55/262a9111-a0c2-4bdb-b21f-e33adb0241de/24e78a99-bad3-4a7d-9156-152997ea8218"
-					(reference "R8")
-					(unit 1)
-				)
-			)
-		)
-	)
+					(reference "R6")
+					(unit 1)
+				)
+			)
+		)
+	)
+	(sheet_instances
+		(path "/"
+			(page "1")
+		)
+	)
+	(embedded_fonts no)
 )
