File: Wsprry Pi Controls/KiCad Design/Wsprry Pi Controls.kicad_sch (KiCad schematic)
At the start: 2 parts, among them SW1 SW_Push

Commit message: Notionally complete through PA
Parts:
- added C1: 0.1µF, Capacitor_SMD:C_0603_1608Metric, symbol Device:C
- added R1: 270Ω, Resistor_SMD:R_0603_1608Metric, symbol Device:R_US
- added R2: 10kΩ, Resistor_SMD:R_0603_1608Metric, symbol Device:R_US
- D1: value LED -> RED; footprint (none) -> LED_SMD:LED_0603_1608Metric
- SW1: footprint (none) -> Button_Switch_SMD:SW_Push_1TS009xxxx-xxxx-xxxx_6x6x5mm
Connections:
- net GPIO_SHUTDOWN: now also C1.1, R2.2
- net GPIO_TXLED: now also R1.2; no longer D1.2 (A)
- net SHUTDOWN_GND: now also C1.2
- new net: D1.2 (A), R1.1
- new net SHUTDOWN_3V3: R2.1
Other:
- note removed: "Wsprry Pi External Controls"
- title: Wsprry Pi External Controls -> Wsprry Pi Controls
- moved on the sheet: D1, SW1
