File: Wsprry Pi µHAT/KiCad Design/Wsprry_Pi_uHAT.kicad_pcb (KiCad board)
At the start: 2 copper layers, 65 x 30 mm, 10 parts, among them J1 GPIO, U2 CAT24C128

Commit message: Notionally complete through PA
Parts:
- removed JP1: ID_WP, Jumper:SolderJumper-2_P1.3mm_Open_RoundedPad1.0x1.5mm
- added C10: 0.1µF, Capacitor_SMD:C_0603_1608Metric, F.Cu at (135.1, 91.5)
- added C11: 1µF, Capacitor_SMD:C_0603_1608Metric, F.Cu at (132.8, 94.3)
- added C12: 10µF, Capacitor_SMD:C_1206_3216Metric, F.Cu at (138.5, 91.1)
- added C13: 0.1F, Capacitor_SMD:C_0603_1608Metric, F.Cu at (145.4, 91.9)
- added C14: 100n, Capacitor_SMD:C_0603_1608Metric, F.Cu at (147.8, 83.5)
- added C15: 22nF, Capacitor_SMD:C_0603_1608Metric, F.Cu at (129.2, 94.3)
- added C16: 22pF, Capacitor_SMD:C_0603_1608Metric, F.Cu at (125.5, 87.6)
- added C17: 100pF, Capacitor_SMD:C_0603_1608Metric, F.Cu at (126.0, 81.2)
- added C18: 10µF, Capacitor_SMD:C_1210_3225Metric, F.Cu at (134.2, 83.4)
- added C19: 1.0µF, Capacitor_SMD:C_0805_2012Metric, F.Cu at (131.6, 82.9)
- added C2: 0.1uF, Capacitor_SMD:C_0603_1608Metric, F.Cu at (163.0, 89.2)
- added C20: 0.1µF, Capacitor_SMD:C_0603_1608Metric, F.Cu at (129.9, 82.7)
- added C3: 1.0uF, Capacitor_SMD:C_0603_1608Metric, F.Cu at (163.0, 87.7)
- added C4: 1nF, Capacitor_SMD:C_0603_1608Metric, F.Cu at (158.4, 88.3)
- added C5: 0.1µF, Capacitor_SMD:C_0603_1608Metric, F.Cu at (150.9, 93.3)
- added C6: 1.0µF, Capacitor_SMD:C_0603_1608Metric, F.Cu at (148.5, 86.9)
- added C7: 0.1µF, Capacitor_SMD:C_0603_1608Metric, F.Cu at (148.0, 93.3)
- added C8: 1uF, Capacitor_SMD:C_0603_1608Metric, F.Cu at (140.1, 98.1)
- added C9: 1.0µF, Capacitor_SMD:C_0603_1608Metric, F.Cu at (136.6, 91.5)
- added D1: RED, LED_SMD:LED_0603_1608Metric, F.Cu at (115.3, 77.3)
- added D2: BAT54J, Diode_SMD:D_SOD-323F, F.Cu at (128.7, 92.0)
- added D3: 5.1V, Diode_SMD:D_SOD-123, F.Cu at (124.2, 90.9)
- added FB1: 600Ω@100MHz, Inductor_SMD:L_0603_1608Metric, F.Cu at (163.0, 86.3)
- added FB2: 600Ω@100MHz, Inductor_SMD:L_0603_1608Metric, F.Cu at (149.5, 93.3)
- added FB3: 600Ω100MHz, Inductor_SMD:L_0805_2012Metric, F.Cu at (140.5, 91.5)
- added FB4: 600Ω@100MHZ, Inductor_SMD:L_0603_1608Metric, F.Cu at (136.5, 82.7)
- added L1: 2.2µH, Inductor_SMD:L_0805_2012Metric, F.Cu at (133.6, 91.8)
- added L2: 2.2µH, Inductor_SMD:L_1206_3216Metric, F.Cu at (127.9, 83.5)
- added Q1: AO3400A, Package_TO_SOT_SMD:SOT-23, F.Cu at (128.0, 87.8)
- added R10: 292Ω, Resistor_SMD:R_0603_1608Metric, F.Cu at (143.2, 95.6)
- added R11: 47kΩ, Resistor_SMD:R_0603_1608Metric, F.Cu at (146.3, 80.5)
- added R12: 3.9K, Resistor_SMD:R_0603_1608Metric, F.Cu at (152.0, 83.6)
- added R13: 0Ω, Resistor_SMD:R_0603_1608Metric, F.Cu at (146.3, 83.5)
- added R14: 3.9K, Resistor_SMD:R_0603_1608Metric, F.Cu at (150.6, 83.6)
- added R15: 49.9Ω, Resistor_SMD:R_0603_1608Metric, F.Cu at (124.8, 94.3)
- added R16: 10Ω, Resistor_SMD:R_0603_1608Metric, F.Cu at (127.0, 93.5)
- added R17: 100Ω, Resistor_SMD:R_0603_1608Metric, F.Cu at (126.0, 84.2)
- added R3: 33Ω, Resistor_SMD:R_0603_1608Metric, F.Cu at (158.4, 91.3)
- added R4: 0Ω, Resistor_SMD:R_0603_1608Metric, F.Cu at (157.0, 88.4)
- added R5: 2K2, Resistor_SMD:R_0603_1608Metric, F.Cu at (151.2, 86.2)
- added R6: 2K2, Resistor_SMD:R_0603_1608Metric, F.Cu at (151.2, 87.6)
- added R7: 0Ω, Resistor_SMD:R_0603_1608Metric, F.Cu at (140.1, 95.1)
- added R8: 292Ω, Resistor_SMD:R_0603_1608Metric, F.Cu at (143.2, 94.0)
- added R9: 17.6Ω, Resistor_SMD:R_0603_1608Metric, F.Cu at (145.4, 94.8)
- added SW1: SW_Push, Button_Switch_SMD:SW_Push_1TS009xxxx-xxxx-xxxx_6x6x5mm, F.Cu at (160.7, 79.9)
- added TP1: TP_XRAW, TestPoint:TestPoint_2Pads_Pitch2.54mm_Drill0.8mm, F.Cu at (160.3, 92.1)
- added TP2: TP_XREF, TestPoint:TestPoint_2Pads_Pitch2.54mm_Drill0.8mm, F.Cu at (155.1, 89.6)
- added TP3: TP_PAD_OUT, TestPoint:TestPoint_2Pads_Pitch2.54mm_Drill0.8mm, F.Cu at (143.2, 98.9)
- added TP4: TP_PAOUT, TestPoint:TestPoint_2Pads_Pitch2.54mm_Drill0.8mm, F.Cu at (123.7, 86.8)
- added U1: GVA-84, Package_TO_SOT_SMD:SOT-89-3, F.Cu at (136.9, 96.3)
- added Y1: ATX-11-F-27.000MHZ-F05-T, Oscillator:Oscillator_SMD_SeikoEpson_TG2520SMN-xxx-xxxxxx-4Pin_2.5x2.0mm, F.Cu at (163.0, 91.7)
- added Y2: Si5351A-B-GT, Package_SO:MSOP-10_3x3mm_P0.5mm, F.Cu at (149.5, 90.1)
- C1: value 100n -> 0.1µF; footprint Capacitor_SMD:C_0201_0603Metric -> Capacitor_SMD:C_0603_1608Metric
- J1: value GPIO -> Raspberry Pi Header; footprint Connector_PinSocket_2.54mm:PinSocket_2x20_P2.54mm_Vertical -> Wsprry Pi µHAT+:PinSocket_2x20_P2.54mm_Vertical
- R1: value 3.9K -> 270Ω; footprint Resistor_SMD:R_0201_0603Metric -> Resistor_SMD:R_0603_1608Metric
- R2: value 3.9K -> 10kΩ; footprint Resistor_SMD:R_0201_0603Metric -> Resistor_SMD:R_0603_1608Metric
- U2: value CAT24C128 -> 24LC128; footprint Package_SO:TSSOP-8_4.4x3mm_P0.65mm -> Package_SO:SOIC-8_3.9x4.9mm_P1.27mm
- moved R1 37.0 mm to (118.3, 77.3), turned to 0 degrees
- moved C1 8.98 mm to (155.7, 81.2)
- moved R2 3.43 mm to (155.7, 78.2)
- moved U2 2.28 mm to (150.9, 79.4)
Connections:
- net +5V renamed 5V
- C1 pad 1: +3V3 -> /Raspberry Pi Header/PI_SHUTDOWN
- J1 pad 1: +3V3 -> 3V3
- J1 pad 10: /GPIO15/RXD0 -> unconnected-(J1-GPIO15-Pad10)
- J1 pad 11: /GPIO17 -> unconnected-(J1-GPIO17-Pad11)
- J1 pad 12: /GPIO18/PCM.CLK -> /Raspberry Pi Header/PI_TXLED
- J1 pad 13: /GPIO27 -> unconnected-(J1-GPIO27-Pad13)
- J1 pad 14: GND -> unconnected-(J1-GND-Pad14)
- J1 pad 15: /GPIO22 -> unconnected-(J1-GPIO22-Pad15)
- J1 pad 16: /GPIO23 -> unconnected-(J1-GPIO23-Pad16)
- J1 pad 17: +3V3 -> 3V3
- J1 pad 18: /GPIO24 -> unconnected-(J1-GPIO24-Pad18)
- J1 pad 19: /GPIO10/SPI0.MOSI -> unconnected-(J1-GPIO10-Pad19)
- J1 pad 20: GND -> unconnected-(J1-GND-Pad20)
- J1 pad 21: /GPIO9/SPI0.MISO -> unconnected-(J1-GPIO9-Pad21)
- J1 pad 22: /GPIO25 -> unconnected-(J1-GPIO25-Pad22)
- J1 pad 23: /GPIO11/SPI0.SCLK -> unconnected-(J1-GPIO11-Pad23)
- J1 pad 24: /GPIO8/SPI0.CE0 -> unconnected-(J1-GPIO8-Pad24)
- J1 pad 26: /GPIO7/SPI0.CE1 -> unconnected-(J1-GPIO7-Pad26)
- J1 pad 27: /ID_SDA -> /HAT+ EEPROM/ID_SDA
- J1 pad 28: /ID_SCL -> /HAT+ EEPROM/ID_SCL
- J1 pad 29: /GPIO5 -> unconnected-(J1-GPIO5-Pad29)
- J1 pad 3: /GPIO2/SDA1 -> /Raspberry Pi Header/PI_SDA
- J1 pad 30: GND -> unconnected-(J1-GND-Pad30)
- J1 pad 31: /GPIO6 -> unconnected-(J1-GPIO6-Pad31)
- J1 pad 32: /GPIO12/PWM0 -> unconnected-(J1-GPIO12-Pad32)
- J1 pad 33: /GPIO13/PWM1 -> unconnected-(J1-GPIO13-Pad33)
- J1 pad 34: GND -> unconnected-(J1-GND-Pad34)
- J1 pad 35: /GPIO19/PCM.FS -> /Raspberry Pi Header/PI_SHUTDOWN
- J1 pad 36: /GPIO16 -> unconnected-(J1-GPIO16-Pad36)
- J1 pad 37: /GPIO26 -> unconnected-(J1-GPIO26-Pad37)
- J1 pad 38: /GPIO20/PCM.DIN -> unconnected-(J1-GPIO20-Pad38)
- J1 pad 40: /GPIO21/PCM.DOUT -> unconnected-(J1-GPIO12-Pad40)
- J1 pad 5: /GPIO3/SCL1 -> /Raspberry Pi Header/PI_SCL
- J1 pad 6: GND -> unconnected-(J1-GND-Pad6)
- J1 pad 7: /GPIO4/GPCLK0 -> unconnected-(J1-Pin_7-Pad7)
- J1 pad 8: /GPIO14/TXD0 -> unconnected-(J1-GPIO14-Pad8)
- R1 pad 1: +3V3 -> Net-(D1-A)
- R1 pad 2: /ID_SDA -> /Raspberry Pi Header/PI_TXLED
- R2 pad 1: +3V3 -> 3V3
- R2 pad 2: /ID_SCL -> /Raspberry Pi Header/PI_SHUTDOWN
- U2 pad 1: unconnected-(U2-A0-Pad1) -> GND
- U2 pad 2: unconnected-(U2-A1-Pad2) -> GND
- U2 pad 3: unconnected-(U2-A2-Pad3) -> GND
- U2 pad 5: /ID_SDA -> /HAT+ EEPROM/ID_SDA
- U2 pad 6: /ID_SCL -> /HAT+ EEPROM/ID_SCL
- U2 pad 8: +3V3 -> 3V3
Routing:
- net 3V3: track 0.00 -> 135.8 mm
- net 5V: track 0.00 -> 73.9 mm
- net /Raspberry Pi Header/PI_SCL: track 0.00 -> 56.4 mm
- net /Raspberry Pi Header/PI_SDA: track 0.00 -> 54.6 mm
- net +3V3: track 32.5 -> 0.00 mm
- net /ID_SCL: track 21.6 -> 0.00 mm
- net /HAT+ EEPROM/ID_SCL: track 0.00 -> 19.8 mm
- net /ID_SDA: track 18.6 -> 0.00 mm
- net Net-(Y2-VDD): track 0.00 -> 17.8 mm
- net Net-(D2-A): track 0.00 -> 17.1 mm
- net /HAT+ EEPROM/ID_SDA: track 0.00 -> 16.6 mm
- net /Si5153 Chain/Final PA/PA_OUT: track 0.00 -> 15.9 mm
- net /Raspberry Pi Header/PI_SHUTDOWN: track 0.00 -> 12.0 mm
- net Net-(C18-Pad1): track 0.00 -> 8.57 mm
- net Net-(C10-Pad1): track 0.00 -> 8.32 mm
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- added copper zone on F.Cu, net Net-(D2-A)
Other:
- board text removed: "PoE"
